File: DCSDv2_CP2102N/DCSDv2_CP2102N.kicad_sch (KiCad schematic)
At the start: 18 parts, among them P1 USB_C_Plug_USB2.0, U1 CP2102N-Axx-xQFN28

Commit message: Version 1.1
Parts:
- JP1, JP2: footprint Jumper:SolderJumper-2_P1.3mm_Bridged_RoundedPad1.0x1.5mm -> Jumper:SolderJumper-2_P1.3mm_Open_RoundedPad1.0x1.5mm; symbol Jumper:SolderJumper_2_Bridged -> Jumper:SolderJumper_2_Open
Connections:
- net DC_CTS: now also U2.6 (RTS); no longer U2.7 (CTS)
- net DC_RTS: now also U2.7 (CTS); no longer U2.6 (RTS)
- net DC_RX: now also U2.5 (TX); no longer U2.4 (RX)
- net DC_TX: now also U2.4 (RX); no longer U2.5 (TX)
Changed lines of the file:
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@@
     (effects (font (size 1.27 1.27)) (justify right bottom))
   )
-  (label "DC_RTS" (at 168.402 60.198 180) (fields_autoplaced)
+  (label "DC_RTS" (at 168.402 57.658 180) (fields_autoplaced)
     (effects (font (size 1.27 1.27)) (justify right bottom))
   )
@@
     (effects (font (size 1.27 1.27)) (justify right bottom))
   )
-  (label "DC_TX" (at 168.402 62.738 180) (fields_autoplaced)
+  (label "DC_TX" (at 168.402 65.278 180) (fields_autoplaced)
     (effects (font (size 1.27 1.27)) (justify right bottom))
   )
@@
     (effects (font (size 1.27 1.27)) (justify left bottom))
   )
-  (label "DC_CTS" (at 168.402 57.658 180) (fields_autoplaced)
+  (label "DC_CTS" (at 168.402 60.198 180) (fields_autoplaced)
     (effects (font (size 1.27 1.27)) (justify right bottom))
   )
@@
     (effects (font (size 1.27 1.27)) (justify right bottom))
   )
-  (label "DC_RX" (at 168.402 65.278 180) (fields_autoplaced)
+  (label "DC_RX" (at 168.402 62.738 180) (fields_autoplaced)
     (effects (font (size 1.27 1.27)) (justify right bottom))
   )
@@
     )
   )
-  (symbol (lib_id "Jumper:SolderJumper_2_Bridged") (at 116.078 22.098 0) (unit 1)
+  (symbol (lib_id "Jumper:SolderJumper_2_Open") (at 116.078 22.098 0) (unit 1)
     (in_bom yes) (on_board yes) (dnp no) (fields_autoplaced)
     (property "Reference" "JP1" (at 116.078 16.51 0)
@@
       (effects (font (size 1.27 1.27)))
     )
-    (property "Footprint" "Jumper:SolderJumper-2_P1.3mm_Bridged_RoundedPad1.0x1.5mm" (at 116.078 22.098 0)
+    (property "Footprint" "Jumper:SolderJumper-2_P1.3mm_Open_RoundedPad1.0x1.5mm" (at 116.078 22.098 0)
       (effects (font (size 1.27 1.27)) hide)
     )
@@
     )
   )
-  (symbol (lib_id "Jumper:SolderJumper_2_Bridged") (at 116.078 31.496 0) (unit 1)
+  (symbol (lib_id "Jumper:SolderJumper_2_Open") (at 116.078 31.496 0) (unit 1)
     (in_bom yes) (on_board yes) (dnp no) (fields_autoplaced)
     (property "Reference" "JP2" (at 116.078 25.908 0)
@@
       (effects (font (size 1.27 1.27)))
     )
-    (property "Footprint" "Jumper:SolderJumper-2_P1.3mm_Bridged_RoundedPad1.0x1.5mm" (at 116.078 31.496 0)
-      (effects (font (size 1.27 1.27)) hide)
-    )
+    (property "Footprint" "Jumper:SolderJumper-2_P1.3mm_Open_RoundedPad1.0x1.5mm" (at 116.078 31.496 0)
+      (effects (font (size 1.27 1.27)) hide)
+    )
